File: HW5/JDPHW5.kicad_pcb (KiCad board)
At the start: 2 copper layers, 47.5 x 41.8 mm, 16 parts, among them J1 Conn_01x03_Pin, J2 Conn_01x02_Pin, U1 NSL-32, U2 NSL-32, U3 TLV2372

Commit message: Save
Some things still need footprints like the pins but mostly just need to connect things now I believe
Parts:
- added ?: , , F.Cu at (213.4, 73.7)
- added ?: , , F.Cu at (231.1, 53.3)
- added ?: , , F.Cu at (213.4, 61.0)
- added ?: , , F.Cu at (241.3, 91.4)
- added ?: , , F.Cu at (236.2, 99.1)
- added ?: , , F.Cu at (223.5, 99.1)
- added ?: , , F.Cu at (226.1, 83.8)
- added ?: , , F.Cu at (251.5, 86.4)
- added ?: , , F.Cu at (238.8, 78.7)
- added ?: , , F.Cu at (228.6, 91.4)
- added ?: , , F.Cu at (238.8, 91.4)
- added ?: , , F.Cu at (241.3, 99.1)
- added ?: , , F.Cu at (210.8, 99.1)
- added ?: , , F.Cu at (215.9, 53.3)
- added ?: , , F.Cu at (210.8, 88.9)
- added ?: , , F.Cu at (243.8, 68.6)
- added ?: , , F.Cu at (246.4, 53.3)
- added ?: , , F.Cu at (221.0, 86.4)
- added ?: , , F.Cu at (208.3, 73.7)
- added ?: , , F.Cu at (236.2, 73.7)
- added ?: , , F.Cu at (213.4, 58.4)
- added ?: , , F.Cu at (223.5, 83.8)
- added ?: , , F.Cu at (251.5, 88.9)
- added ?: , , F.Cu at (228.6, 71.1)
- added ?: , , F.Cu at (221.0, 94.0)
- added ?: , , F.Cu at (215.9, 66.0)
- added ?: , , F.Cu at (223.5, 78.7)
- added ?: , , F.Cu at (221.0, 71.1)
- added ?: , , F.Cu at (210.8, 78.7)
- added ?: , , F.Cu at (203.2, 78.7)
- added ?: , , F.Cu at (251.5, 94.0)
- added ?: , , F.Cu at (205.7, 66.0)
- added ?: , , F.Cu at (223.5, 58.4)
- added ?: , , F.Cu at (241.3, 53.3)
- added ?: , , F.Cu at (251.5, 66.0)
- added ?: , , F.Cu at (228.6, 58.4)
- added ?: , , F.Cu at (208.3, 83.8)
- added ?: , , F.Cu at (213.4, 53.3)
- added ?: , , F.Cu at (226.1, 76.2)
- added ?: , , F.Cu at (246.4, 94.0)
- added ?: , , F.Cu at (205.7, 53.3)
- added ?: , , F.Cu at (241.3, 63.5)
- added ?: , , F.Cu at (205.7, 71.1)
- added ?: , , F.Cu at (203.2, 63.5)
- added ?: , , F.Cu at (233.7, 63.5)
- added ?: , , F.Cu at (223.5, 68.6)
- added ?: , , F.Cu at (243.8, 81.3)
- added ?: , , F.Cu at (215.9, 76.2)
- added ?: , , F.Cu at (251.5, 96.5)
- added ?: , , F.Cu at (218.4, 61.0)
- added ?: , , F.Cu at (223.5, 73.7)
- added ?: , , F.Cu at (248.9, 68.6)
- added ?: , , F.Cu at (205.7, 96.5)
- added ?: , , F.Cu at (226.1, 86.4)
- added ?: , , F.Cu at (213.4, 86.4)
- added ?: , , F.Cu at (215.9, 61.0)
- added ?: , , F.Cu at (210.8, 83.8)
- added ?: , , F.Cu at (238.8, 76.2)
- added ?: , , F.Cu at (226.1, 88.9)
- added ?: , , F.Cu at (221.0, 83.8)
- added ?: , , F.Cu at (248.9, 94.0)
- added ?: , , F.Cu at (203.2, 76.2)
- added ?: , , F.Cu at (238.8, 96.5)
- added ?: , , F.Cu at (208.3, 63.5)
- added ?: , , F.Cu at (208.3, 68.6)
- added ?: , , F.Cu at (236.2, 94.0)
- added ?: , , F.Cu at (213.4, 63.5)
- added ?: , , F.Cu at (223.5, 55.9)
- added ?: , , F.Cu at (208.3, 71.1)
- added ?: , , F.Cu at (228.6, 94.0)
- added ?: , , F.Cu at (231.1, 73.7)
- added ?: , , F.Cu at (213.4, 83.8)
- added ?: , , F.Cu at (223.5, 88.9)
- added ?: , , F.Cu at (221.0, 76.2)
- added ?: , , F.Cu at (205.7, 55.9)
- added ?: , , F.Cu at (236.2, 63.5)
- added ?: , , F.Cu at (238.8, 81.3)
- added ?: , , F.Cu at (226.1, 81.3)
- added ?: , , F.Cu at (223.5, 71.1)
- added ?: , , F.Cu at (203.2, 50.8)
- added ?: , , F.Cu at (236.2, 71.1)
- added ?: , , F.Cu at (248.9, 96.5)
- added ?: , , F.Cu at (221.0, 66.0)
- added ?: , , F.Cu at (221.0, 58.4)
- added ?: , , F.Cu at (248.9, 88.9)
- added ?: , , F.Cu at (243.8, 50.8)
- added ?: , , F.Cu at (246.4, 66.0)
- added ?: , , F.Cu at (218.4, 73.7)
- added ?: , , F.Cu at (203.2, 61.0)
- added ?: , , F.Cu at (228.6, 63.5)
- added ?: , , F.Cu at (241.3, 96.5)
- added ?: , , F.Cu at (226.1, 53.3)
- added ?: , , F.Cu at (203.2, 96.5)
- added ?: , , F.Cu at (208.3, 61.0)
- added ?: , , F.Cu at (246.4, 96.5)
- added ?: , , F.Cu at (251.5, 71.1)
- added ?: , , F.Cu at (218.4, 71.1)
- added ?: , , F.Cu at (223.5, 50.8)
- added ?: , , F.Cu at (213.4, 94.0)
- added ?: , , F.Cu at (231.1, 61.0)
- added ?: , , F.Cu at (246.4, 99.1)
- added ?: , , F.Cu at (218.4, 96.5)
- added ?: , , F.Cu at (233.7, 66.0)
- added ?: , , F.Cu at (213.4, 91.4)
- added ?: , , F.Cu at (241.3, 66.0)
- added ?: , , F.Cu at (231.1, 63.5)
- added ?: , , F.Cu at (248.9, 61.0)
- added ?: , , F.Cu at (233.7, 55.9)
- added ?: , , F.Cu at (205.7, 91.4)
- added ?: , , F.Cu at (205.7, 86.4)
- added ?: , , F.Cu at (238.8, 63.5)
- added ?: , , F.Cu at (205.7, 99.1)
- added ?: , , F.Cu at (221.0, 88.9)
- added ?: , , F.Cu at (205.7, 78.7)
- added ?: , , F.Cu at (233.7, 81.3)
- added ?: , , F.Cu at (226.1, 71.1)
- added ?: , , F.Cu at (236.2, 83.8)
- added ?: , , F.Cu at (243.8, 99.1)
- added ?: , , F.Cu at (231.1, 76.2)
- added ?: , , F.Cu at (226.1, 99.1)
- added ?: , , F.Cu at (215.9, 81.3)
- added ?: , , F.Cu at (210.8, 94.0)
- added ?: , , F.Cu at (251.5, 53.3)
- added ?: , , F.Cu at (213.4, 99.1)
- added ?: , , F.Cu at (246.4, 83.8)
- added ?: , , F.Cu at (223.5, 86.4)
- added ?: , , F.Cu at (231.1, 78.7)
- added ?: , , F.Cu at (213.4, 96.5)
- added ?: , , F.Cu at (203.2, 99.1)
- added ?: , , F.Cu at (233.7, 99.1)
- added ?: , , F.Cu at (233.7, 76.2)
- added ?: , , F.Cu at (210.8, 68.6)
- added ?: , , F.Cu at (251.5, 81.3)
- added ?: , , F.Cu at (241.3, 94.0)
- added ?: , , F.Cu at (203.2, 68.6)
- added ?: , , F.Cu at (205.7, 94.0)
- added ?: , , F.Cu at (228.6, 73.7)
- added ?: , , F.Cu at (210.8, 53.3)
- added ?: , , F.Cu at (208.3, 53.3)
- added ?: , , F.Cu at (208.3, 81.3)
- added ?: , , F.Cu at (218.4, 55.9)
- added ?: , , F.Cu at (210.8, 96.5)
- added ?: , , F.Cu at (221.0, 61.0)
- added ?: , , F.Cu at (218.4, 91.4)
- added ?: , , F.Cu at (203.2, 81.3)
- added ?: , , F.Cu at (226.1, 58.4)
- added ?: , , F.Cu at (228.6, 88.9)
- added ?: , , F.Cu at (236.2, 86.4)
- added ?: , , F.Cu at (208.3, 86.4)
- added ?: , , F.Cu at (233.7, 71.1)
- added ?: , , F.Cu at (213.4, 76.2)
- added ?: , , F.Cu at (208.3, 58.4)
- added ?: , , F.Cu at (233.7, 78.7)
- added ?: , , F.Cu at (233.7, 58.4)
- added ?: , , F.Cu at (233.7, 96.5)
- added ?: , , F.Cu at (205.7, 76.2)
- added ?: , , F.Cu at (228.6, 76.2)
- added ?: , , F.Cu at (241.3, 50.8)
- added ?: , , F.Cu at (241.3, 73.7)
- added ?: , , F.Cu at (231.1, 71.1)
- added ?: , , F.Cu at (238.8, 66.0)
- added ?: , , F.Cu at (208.3, 66.0)
- added ?: , , F.Cu at (241.3, 71.1)
- added ?: , , F.Cu at (221.0, 68.6)
- added ?: , , F.Cu at (223.5, 66.0)
- added ?: , , F.Cu at (243.8, 58.4)
- added ?: , , F.Cu at (251.5, 83.8)
- added ?: , , F.Cu at (231.1, 55.9)
- added ?: , , F.Cu at (238.8, 55.9)
- added ?: , , F.Cu at (221.0, 50.8)
- added ?: , , F.Cu at (213.4, 81.3)
- added ?: , , F.Cu at (236.2, 50.8)
- added ?: , , F.Cu at (248.9, 66.0)
- added ?: , , F.Cu at (251.5, 73.7)
- added ?: , , F.Cu at (218.4, 50.8)
- added ?: , , F.Cu at (213.4, 78.7)
- added ?: , , F.Cu at (205.7, 88.9)
- added ?: , , F.Cu at (223.5, 94.0)
- added ?: , , F.Cu at (228.6, 78.7)
- added ?: , , F.Cu at (238.8, 99.1)
- added ?: , , F.Cu at (210.8, 55.9)
- added ?: , , F.Cu at (221.0, 99.1)
- added ?: , , F.Cu at (243.8, 66.0)
- added ?: , , F.Cu at (223.5, 61.0)
- added ?: , , F.Cu at (251.5, 61.0)
- added ?: , , F.Cu at (246.4, 61.0)
- added ?: , , F.Cu at (238.8, 88.9)
- added ?: , , F.Cu at (248.9, 71.1)
- added ?: , , F.Cu at (226.1, 55.9)
- added ?: , , F.Cu at (241.3, 76.2)
- added ?: , , F.Cu at (241.3, 86.4)
- added ?: , , F.Cu at (238.8, 68.6)
- added ?: , , F.Cu at (226.1, 91.4)
- added ?: , , F.Cu at (228.6, 81.3)
- added ?: , , F.Cu at (238.8, 58.4)
- added ?: , , F.Cu at (231.1, 96.5)
- added ?: , , F.Cu at (233.7, 86.4)
- added ?: , , F.Cu at (213.4, 66.0)
- added ?: , , F.Cu at (243.8, 86.4)
- added ?: , , F.Cu at (205.7, 50.8)
- added ?: , , F.Cu at (203.2, 94.0)
- added ?: , , F.Cu at (218.4, 63.5)
- added ?: , , F.Cu at (233.7, 91.4)
- added ?: , , F.Cu at (251.5, 68.6)
- added ?: , , F.Cu at (241.3, 68.6)
- added ?: , , F.Cu at (228.6, 68.6)
- added ?: , , F.Cu at (251.5, 58.4)
- added ?: , , F.Cu at (246.4, 71.1)
- added ?: , , F.Cu at (251.5, 55.9)
- added ?: , , F.Cu at (210.8, 76.2)
- added ?: , , F.Cu at (226.1, 96.5)
- added ?: , , F.Cu at (231.1, 66.0)
- added ?: , , F.Cu at (215.9, 94.0)
- added ?: , , F.Cu at (236.2, 55.9)
- added ?: , , F.Cu at (221.0, 73.7)
- added ?: , , F.Cu at (223.5, 91.4)
- added ?: , , F.Cu at (236.2, 88.9)
- added ?: , , F.Cu at (243.8, 78.7)
- added ?: , , F.Cu at (236.2, 66.0)
- added ?: , , F.Cu at (210.8, 58.4)
- added ?: , , F.Cu at (236.2, 81.3)
- added ?: , , F.Cu at (205.7, 61.0)
- added ?: , , F.Cu at (215.9, 91.4)
- added ?: , , F.Cu at (236.2, 53.3)
- added ?: , , F.Cu at (248.9, 58.4)
- added ?: , , F.Cu at (251.5, 76.2)
- added ?: , , F.Cu at (246.4, 50.8)
- added ?: , , F.Cu at (203.2, 86.4)
- added ?: , , F.Cu at (241.3, 81.3)
- added ?: , , F.Cu at (221.0, 63.5)
- added ?: , , F.Cu at (205.7, 58.4)
- added ?: , , F.Cu at (248.9, 99.1)
- added ?: , , F.Cu at (226.1, 68.6)
- added ?: , , F.Cu at (233.7, 68.6)
- added ?: , , F.Cu at (248.9, 73.7)
- added ?: , , F.Cu at (228.6, 53.3)
- added ?: , , F.Cu at (221.0, 81.3)
- added ?: , , F.Cu at (215.9, 58.4)
- added ?: , , F.Cu at (226.1, 78.7)
- added ?: , , F.Cu at (236.2, 91.4)
- added ?: , , F.Cu at (243.8, 61.0)
- added ?: , , F.Cu at (215.9, 55.9)
- added ?: , , F.Cu at (231.1, 58.4)
- added ?: , , F.Cu at (243.8, 76.2)
- added ?: , , F.Cu at (218.4, 86.4)
- added ?: , , F.Cu at (246.4, 73.7)
- added ?: , , F.Cu at (236.2, 68.6)
- added ?: , , F.Cu at (208.3, 50.8)
- added ?: , , F.Cu at (233.7, 88.9)
- added ?: , , F.Cu at (233.7, 94.0)
- added ?: , , F.Cu at (228.6, 61.0)
- added ?: , , F.Cu at (243.8, 53.3)
- added ?: , , F.Cu at (215.9, 68.6)
- added ?: , , F.Cu at (231.1, 68.6)
- added ?: , , F.Cu at (236.2, 61.0)
- added ?: , , F.Cu at (223.5, 63.5)
- added ?: , , F.Cu at (226.1, 73.7)
- added ?: , , F.Cu at (238.8, 94.0)
- added ?: , , F.Cu at (215.9, 96.5)
- added ?: , , F.Cu at (221.0, 53.3)
- added ?: , , F.Cu at (223.5, 53.3)
- added ?: , , F.Cu at (208.3, 94.0)
- added ?: , , F.Cu at (215.9, 99.1)
- added ?: , , F.Cu at (218.4, 94.0)
- added ?: , , F.Cu at (231.1, 91.4)
- added ?: , , F.Cu at (215.9, 86.4)
- added ?: , , F.Cu at (210.8, 61.0)
- added ?: , , F.Cu at (213.4, 55.9)
- added ?: , , F.Cu at (210.8, 91.4)
- added ?: , , F.Cu at (243.8, 73.7)
- added ?: , , F.Cu at (243.8, 94.0)
- added ?: , , F.Cu at (223.5, 96.5)
- added ?: , , F.Cu at (248.9, 50.8)
- added ?: , , F.Cu at (248.9, 55.9)
- added ?: , , F.Cu at (213.4, 68.6)
- added ?: , , F.Cu at (215.9, 78.7)
- added ?: , , F.Cu at (215.9, 83.8)
- added ?: , , F.Cu at (218.4, 78.7)
- added ?: , , F.Cu at (241.3, 78.7)
- added ?: , , F.Cu at (231.1, 94.0)
- added ?: , , F.Cu at (208.3, 78.7)
- added ?: , , F.Cu at (203.2, 53.3)
- added ?: , , F.Cu at (248.9, 83.8)
- added ?: , , F.Cu at (228.6, 55.9)
- added ?: , , F.Cu at (210.8, 71.1)
- added ?: , , F.Cu at (203.2, 88.9)
- added ?: , , F.Cu at (231.1, 50.8)
- added ?: , , F.Cu at (243.8, 91.4)
- added ?: , , F.Cu at (233.7, 50.8)
- added ?: , , F.Cu at (210.8, 86.4)
- added ?: , , F.Cu at (231.1, 81.3)
- added ?: , , F.Cu at (248.9, 76.2)
- added ?: , , F.Cu at (246.4, 86.4)
- added ?: , , F.Cu at (203.2, 73.7)
- added ?: , , F.Cu at (238.8, 61.0)
- added ?: , , F.Cu at (208.3, 88.9)
- added ?: , , F.Cu at (203.2, 91.4)
- added ?: , , F.Cu at (248.9, 53.3)
- added ?: , , F.Cu at (251.5, 63.5)
- added ?: , , F.Cu at (246.4, 91.4)
- added ?: , , F.Cu at (226.1, 66.0)
- added ?: , , F.Cu at (243.8, 71.1)
- added ?: , , F.Cu at (251.5, 78.7)
- added ?: , , F.Cu at (248.9, 63.5)
- added ?: , , F.Cu at (238.8, 50.8)
- added ?: , , F.Cu at (218.4, 76.2)
- added ?: , , F.Cu at (251.5, 99.1)
- added ?: , , F.Cu at (228.6, 50.8)
- added ?: , , F.Cu at (236.2, 58.4)
- added ?: , , F.Cu at (210.8, 73.7)
- added ?: , , F.Cu at (213.4, 71.1)
- added ?: , , F.Cu at (213.4, 50.8)
- added ?: , , F.Cu at (210.8, 81.3)
- added ?: , , F.Cu at (243.8, 55.9)
- added ?: , , F.Cu at (248.9, 86.4)
- added ?: , , F.Cu at (231.1, 83.8)
- added ?: , , F.Cu at (246.4, 78.7)
- added ?: , , F.Cu at (226.1, 61.0)
- added ?: , , F.Cu at (208.3, 55.9)
- added ?: , , F.Cu at (223.5, 81.3)
- added ?: , , F.Cu at (236.2, 76.2)
- added ?: , , F.Cu at (241.3, 55.9)
- added ?: , , F.Cu at (203.2, 55.9)
- added ?: , , F.Cu at (210.8, 66.0)
- added ?: , , F.Cu at (228.6, 96.5)
- added ?: , , F.Cu at (241.3, 61.0)
- added ?: , , F.Cu at (251.5, 50.8)
- added ?: , , F.Cu at (241.3, 83.8)
- added ?: , , F.Cu at (233.7, 73.7)
- added ?: , , F.Cu at (215.9, 50.8)
- added ?: , , F.Cu at (210.8, 50.8)
- added ?: , , F.Cu at (208.3, 96.5)
- added ?: , , F.Cu at (215.9, 63.5)
- added ?: , , F.Cu at (246.4, 63.5)
- added ?: , , F.Cu at (238.8, 73.7)
- added ?: , , F.Cu at (203.2, 83.8)
- added ?: , , F.Cu at (218.4, 88.9)
- added ?: , , F.Cu at (205.7, 63.5)
- added ?: , , F.Cu at (203.2, 71.1)
- added ?: , , F.Cu at (236.2, 96.5)
- added ?: , , F.Cu at (226.1, 94.0)
- added ?: , , F.Cu at (203.2, 66.0)
- added ?: , , F.Cu at (228.6, 86.4)
- added ?: , , F.Cu at (205.7, 81.3)
- added ?: , , F.Cu at (226.1, 63.5)
- added ?: , , F.Cu at (210.8, 63.5)
- added ?: , , F.Cu at (218.4, 66.0)
- added ?: , , F.Cu at (236.2, 78.7)
- added ?: , , F.Cu at (238.8, 71.1)
- added ?: , , F.Cu at (221.0, 55.9)
- added ?: , , F.Cu at (243.8, 96.5)
- added ?: , , F.Cu at (246.4, 55.9)
- added ?: , , F.Cu at (248.9, 91.4)
- added ?: , , F.Cu at (248.9, 81.3)
- added ?: , , F.Cu at (223.5, 76.2)
- added ?: , , F.Cu at (208.3, 99.1)
- added ?: , , F.Cu at (231.1, 99.1)
- added ?: , , F.Cu at (233.7, 53.3)
- added ?: , , F.Cu at (218.4, 53.3)
- added ?: , , F.Cu at (246.4, 58.4)
- added ?: , , F.Cu at (246.4, 88.9)
- added ?: , , F.Cu at (205.7, 83.8)
- added ?: , , F.Cu at (228.6, 99.1)
- added ?: , , F.Cu at (231.1, 86.4)
- added ?: , , F.Cu at (241.3, 58.4)
- added ?: , , F.Cu at (218.4, 68.6)
- added ?: , , F.Cu at (243.8, 88.9)
- added ?: , , F.Cu at (238.8, 53.3)
- added ?: , , F.Cu at (215.9, 71.1)
- added ?: , , F.Cu at (238.8, 83.8)
- added ?: , , F.Cu at (248.9, 78.7)
- added ?: , , F.Cu at (246.4, 76.2)
- added ?: , , F.Cu at (208.3, 91.4)
- added ?: , , F.Cu at (233.7, 61.0)
- added ?: , , F.Cu at (213.4, 88.9)
- added ?: , , F.Cu at (226.1, 50.8)
- added ?: , , F.Cu at (221.0, 96.5)
- added ?: , , F.Cu at (243.8, 83.8)
- added ?: , , F.Cu at (218.4, 83.8)
- added ?: , , F.Cu at (228.6, 66.0)
- added ?: , , F.Cu at (243.8, 63.5)
- added ?: , , F.Cu at (218.4, 99.1)
- added ?: , , F.Cu at (251.5, 91.4)
- added ?: , , F.Cu at (221.0, 78.7)
- added ?: , , F.Cu at (228.6, 83.8)
- added ?: , , F.Cu at (215.9, 73.7)
- added ?: , , F.Cu at (218.4, 58.4)
- added ?: , , F.Cu at (246.4, 81.3)
- added ?: , , F.Cu at (205.7, 68.6)
- added ?: , , F.Cu at (215.9, 88.9)
- added ?: , , F.Cu at (241.3, 88.9)
- added ?: , , F.Cu at (208.3, 76.2)
- added ?: , , F.Cu at (221.0, 91.4)
- added ?: , , F.Cu at (233.7, 83.8)
- added ?: , , F.Cu at (238.8, 86.4)
- added ?: , , F.Cu at (231.1, 88.9)
- added ?: , , F.Cu at (203.2, 58.4)
- added ?: , , F.Cu at (218.4, 81.3)
- added ?: , , F.Cu at (205.7, 73.7)
- added ?: , , F.Cu at (246.4, 68.6)
Routing:
- net (no net): track 0.00 -> 96.5 mm

Commit message: PCB and Sch
Files done
Parts:
- added Inputs1: Conn_01x05, Connector_PinHeader_2.54mm:PinHeader_1x05_P2.54mm_Vertical, F.Cu at (88.9, 144.8)
- added LineOutAudio1: Conn_01x02, Connector_PinHeader_2.54mm:PinHeader_1x02_P2.54mm_Vertical, F.Cu at (135.1, 136.9)
- added Outputs1: Conn_01x05, Connector_PinHeader_2.54mm:PinHeader_1x05_P2.54mm_Vertical, F.Cu at (144.8, 144.8)
- moved ? 115.8 mm to (136.7, 101.6)
- moved ? 115.8 mm to (136.7, 104.1)
- moved ? 115.8 mm to (136.7, 109.2)
- moved ? 115.8 mm to (136.7, 81.3)
- moved ? 115.8 mm to (136.7, 111.8)
- moved ? 115.8 mm to (136.7, 86.4)
- moved ? 115.8 mm to (136.7, 68.6)
- moved ? 115.8 mm to (136.7, 96.5)
- moved ? 115.8 mm to (136.7, 99.1)
- moved ? 115.8 mm to (136.7, 88.9)
- moved ? 115.8 mm to (136.7, 76.2)
- moved ? 115.8 mm to (136.7, 83.8)
- moved ? 115.8 mm to (136.7, 73.7)
- moved ? 115.8 mm to (136.7, 71.1)
- moved ? 115.8 mm to (136.7, 91.4)
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Connections:
- ? pad 1: (no net) -> GND (x20)
- ? pad 1: (no net) -> +3V3 (x20)
- C1 pad 1: unconnected-(C1-Pad1) -> /Audio In 1 (mono)
- C6 pad 1: VCC -> +3V3
- C7 pad 1: VCC -> +3V3
- J2 pad 1: /+3V3 -> +3V3
- R1 pad 1: VCC -> +3V3
- U3 pad 4: unconnected-(U3C-V--Pad4) -> GND
- U3 pad 5: unconnected-(U3B-+-Pad5) -> /U3B_IN+
- U3 pad 6: unconnected-(U3B---Pad6) -> /U3B_IN-
- U3 pad 7: unconnected-(U3-Pad7) -> /U3B_OUT
- U3 pad 8: unconnected-(U3C-V+-Pad8) -> +3V3
Routing:
- net +3V3: track 0.00 -> 221.9 mm
- net GND: track 67.6 -> 179.7 mm
- net (no net): track 96.5 -> 0.00 mm
- net Net-(U3A-+): track 44.4 -> 72.1 mm
- net /Adafruit_2130_A+: track 0.00 -> 22.0 mm, vias 0 -> 1
- net Net-(C1-Pad2): track 53.5 -> 31.8 mm
- net VCC: track 21.2 -> 0.00 mm
- net /Audio In 1 (mono): track 0.00 -> 18.5 mm
- net Net-(C3-Pad1): track 33.6 -> 17.8 mm
- net /PWM2: track 0.06 -> 14.0 mm
- net /U3B_IN+: track 0.00 -> 9.99 mm
- net /U3B_OUT: track 0.00 -> 8.34 mm
- net /U3B_IN-: track 0.00 -> 7.29 mm
- net /PWM1: track 0.00 -> 5.62 mm
- net Net-(U1-A): track 9.29 -> 13.5 mm
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- added copper zone on B.Cu, net GND
- removed copper zone on B.Cu, net VCC
Other:
- board size 47.5 x 41.8 mm -> 63 x 96.5 mm
