File: HW5/JDPHW5.kicad_sch (KiCad schematic)
At the start: 14 parts, among them U1 NSL-32, U2 NSL-32, U3 TLV2372

Commit message: Forgot to save
saved
Parts:
- added unit 2 of U3
- added unit 3 of U3
Connections:
- net at C3.2, C4.1: now also C2.1, U2.3 (R), U3.1, U3.2 (-), U3.3 (+)
Other:
- moved on the sheet: C3, C4, R1

Commit message: Schematic Done
Should be done now with schematic
Parts:
- added J1: Conn_01x03_Pin, Connector_PinHeader_2.54mm:PinHeader_1x03_P2.54mm_Vertical, symbol Connector:Conn_01x03_Pin
- added J2: Conn_01x02_Pin, Connector_PinHeader_2.54mm:PinHeader_1x02_P2.54mm_Vertical, symbol Connector:Conn_01x02_Pin
- U3: footprint (none) -> Package_DIP:DIP-8_W7.62mm
- renumbered R_Volume to R_Volume1
Connections:
- net GND: now also U3.4 (V-), J2.2 (Pin_2)
- net U3B_IN+: now reaches U3.5 (+)
- net U3B_IN+: now also J1.2 (Pin_2)
- net U3B_IN-: now reaches U3.6 (-)
- net U3B_IN-: now also J1.1 (Pin_1)
- net U3B_OUT: now reaches U3.7
- net U3B_OUT: now also J1.3 (Pin_3)
- net PWM2: now reaches R4.1
- net +3V3: now reaches U3.8 (V+)
- net +3V3: now also J2.1 (Pin_1)
- net Adafruit_2130_A+: now reaches R_Volume1.2
- net Audio_In: now reaches C1.1
- net PWM1: now reaches R3.1
- no-connect marks 0 -> 9
Other:
- title: (none) -> HW05 DIY DJ DECK LFP
