File: HW5/JDPHW5.kicad_sch (KiCad schematic)
At the start: 16 parts, among them J1 Conn_01x03_Pin, J2 Conn_01x02_Pin, U1 NSL-32, U2 NSL-32, U3 TLV2372

Commit message: Save
Some things still need footprints like the pins but mostly just need to connect things now I believe
Parts:
- added J4, Outputs: Conn_01x05, symbol Connector_Generic:Conn_01x05
- added LineOutAudio: Conn_01x02, symbol Connector_Generic:Conn_01x02
Connections:
- net GND: now also J4.1 (Pin_1)
- net PWM1: now also J4.4 (Pin_4)
- net PWM2: now also J4.3 (Pin_3)
- new net +3.3V: J4.2 (Pin_2)
- new net Audio In 1 (mono): J4.5 (Pin_5)
- no-connect marks 9 -> 7
Other:
- note added: "In parallel with signal going to Adafruit 2130. R_Volume wiper signal is being sent to the Adafruit 2130 2.5 watt audio amplifier as well as the LineOutAudio connector"
- note added: "Must be on left side of PCB"

Commit message: PCB and Sch
Files done
Parts:
- Inputs1: renamed from J4; footprint (none) -> Connector_PinHeader_2.54mm:PinHeader_1x05_P2.54mm_Vertical
- LineOutAudio1: renamed from LineOutAudio; footprint (none) -> Connector_PinHeader_2.54mm:PinHeader_1x02_P2.54mm_Vertical
- Outputs1: renamed from Outputs; footprint (none) -> Connector_PinHeader_2.54mm:PinHeader_1x05_P2.54mm_Vertical
Connections:
- net +3.3V is gone; now on net +3V3: Inputs1.2 (Pin_2)
- net Audio_In is gone; now on net Audio In 1 (mono): C1.1
- net VCC is gone; now on net +3V3: C6.1, C7.1, R1.1
- net Adafruit_2130_A+: now also LineOutAudio1.1 (Pin_1), LineOutAudio1.2 (Pin_2), Outputs1.3 (Pin_3)
- net GND: now also Outputs1.1 (Pin_1)
- net SD: now reaches Outputs1.2 (Pin_2)
- net A-: now reaches Outputs1.4 (Pin_4)
- net A+: now reaches Outputs1.5 (Pin_5)
- no-connect marks 7 -> 9
Other:
- note removed: "In parallel with signal going to Adafruit 2130. R_Volume wiper signal is being sent to the Adafruit 2130 2.5 watt audio amplifier as well as the LineOutAudio connector"
- moved on the sheet: LineOutAudio1, Outputs1
